File: schematic/power/power.sch (KiCad schematic (older format))
At the start: 14 parts

Commit message: minor in power schematic
Parts:
- added J? (x12): Conn_01x02_Male, symbol Conn_01x02_Male
- added J? (x3): Screw_Terminal_01x02, symbol Screw_Terminal_01x02
Connections:
- net Vdd_12v: now also J?.1 (Pin_1), J?.1 (Pin_1), J?.1 (Pin_1), J?.2 (Pin_2), J?.2 (Pin_2), J?.2 (Pin_2)
- net Vss: now also J?.1 (Pin_1), J?.1 (Pin_1), J?.1 (Pin_1), J?.1 (Pin_1), J?.1 (Pin_1), J?.1 (Pin_1), J?.1 (Pin_1), J?.1 (Pin_1), J?.2 (Pin_2), J?.2 (Pin_2), J?.2 (Pin_2), J?.2 (Pin_2), J?.2 (Pin_2), J?.2 (Pin_2), J?.2 (Pin_2)
- new net 5v_display: J?.1 (Pin_1), J?.2 (Pin_2)
- new net 5v_hub: J?.2 (Pin_2)
- new net 5v_rpi: J?.1 (Pin_1), J?.1 (Pin_1), J?.1 (Pin_1), J?.2 (Pin_2), J?.2 (Pin_2)
Other:
- note added: "Buck Converter\nMP1584"
- moved on the sheet: C?, D?, J?, Q?, R?
