File: schematic/raspi/raspi.sch (KiCad schematic (older format))
At the start: 41 parts

Commit message: ok, lets go again
Connections:
- net disp_button: now reaches J?.11 (GPIO17_(GEN0))
Changed lines of the file:
@@
 Text Notes 10650 7650 0    60   ~ 0
 2
+Text GLabel 4200 3350 0    60   Input ~ 0
+disp_button
+Wire Wire Line
+	4200 3350 4450 3350
 $EndSCHEMATC
