File: schematic/car-control/car-control.kicad_pcb (KiCad board)
At the start: 2 copper layers, 116.1 x 85.3 mm, 49 parts, among them J1 RGBW Sitzbank, J10 Misc Conn, J2 RGBW Hutablage, J3 RPi Front #1, J4 RPi Front #2, J5 Touch Panel, J6 Alarm Control, J7 RGBW Universell 1, J8 Power_Conn, J9 Sig_in_out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

Commit message: i really have no glue what i have done since the last checkin
Parts:
- removed D1: red, led:LED_D5.0mm_Clear
- removed D2: green, led:LED_D5.0mm_Clear
- removed D3: blue, led:LED_D5.0mm_Clear
- removed D4: white, led:LED_D5.0mm_Clear
- removed D5: act_eis, led:LED_D5.0mm_Clear
- removed D7: act_5v, led:LED_D5.0mm_Clear
- removed the REF** at (96.5, 83.6)
- removed the REF** at (200.2, 68.8)
- removed the REF** at (200.2, 140.5)
- removed the REF** at (91.9, 140.5)
- removed the REF** at (179.8, 81.3)
- removed the REF** at (145.5, 125.2)
- added 5v: act_5v, led:LED_D3.0mm_Clear, F.Cu at (100.1, 125.7)
- added J11: Sig_out, TerminalBlock_Phoenix:TerminalBlock_Phoenix_MKDS-1,5-4-5.08_1x04_P5.08mm_Horizontal, F.Cu at (100.8, 141.0)
- added R19: 220, Resistor_THT:R_Axial_DIN0207_L6.3mm_D2.5mm_P10.16mm_Horizontal, F.Cu at (181.4, 83.6)
- added R20: 220, Resistor_THT:R_Axial_DIN0207_L6.3mm_D2.5mm_P10.16mm_Horizontal, F.Cu at (102.6, 131.1)
- added R21: 220, Resistor_THT:R_Axial_DIN0207_L6.3mm_D2.5mm_P10.16mm_Horizontal, F.Cu at (123.4, 121.9)
- added R22: 220, Resistor_THT:R_Axial_DIN0207_L6.3mm_D2.5mm_P10.16mm_Horizontal, F.Cu at (115.6, 106.4)
- added REF**: MountingHole_3.2mm_M3_Pad, MountingHole:MountingHole_3.2mm_M3_Pad, F.Cu at (142.2, 127.8)
- added REF**: MountingHole_3.2mm_M3_Pad, MountingHole:MountingHole_3.2mm_M3_Pad, F.Cu at (199.4, 142.7)
- added REF**: MountingHole_3.2mm_M3_Pad, MountingHole:MountingHole_3.2mm_M3_Pad, F.Cu at (93.5, 140.5)
- added REF**: MountingHole_3.2mm_M3_Pad, MountingHole:MountingHole_3.2mm_M3_Pad, F.Cu at (103.9, 83.6)
- added REF**: MountingHole_3.2mm_M3_Pad, MountingHole:MountingHole_3.2mm_M3_Pad, F.Cu at (199.6, 66.5)
- added blue: blue, led:LED_D3.0mm_Clear, F.Cu at (160.8, 128.8)
- added eis: act_eis, led:LED_D3.0mm_Clear, F.Cu at (131.6, 125.7)
- added green: green, led:LED_D3.0mm_Clear, F.Cu at (189.7, 128.8)
- added horn: horn, led:LED_D3.0mm_Clear, F.Cu at (178.6, 79.8)
- added lock: lock, led:LED_D3.0mm_Clear, F.Cu at (123.4, 127.0)
- added radio: radio, led:LED_D3.0mm_Clear, F.Cu at (159.8, 79.8)
- added red: red, led:LED_D3.0mm_Clear, F.Cu at (170.4, 128.8)
- added unlock: unlock, led:LED_D3.0mm_Clear, F.Cu at (111.8, 108.5)
- added white: white, led:LED_D3.0mm_Clear, F.Cu at (180.1, 128.8)
- J9: value Sig_in_out -> Sig_in; footprint TerminalBlock_Phoenix:TerminalBlock_Phoenix_MKDS-1,5-8-5.08_1x08_P5.08mm_Horizontal -> TerminalBlock_Phoenix:TerminalBlock_Phoenix_MKDS-1,5-2-5.08_1x02_P5.08mm_Horizontal
- moved R18 79.9 mm to (166.9, 83.6)
- moved J9 25.7 mm to (126.5, 141.2)
- moved Q6 3.05 mm to (110.5, 128.5)
- moved R10 3.05 mm to (118.1, 131.6)
Connections:
- A1 pad 14: /sig_220v -> /sig_unlock
- A1 pad 18: Net-(A1-Pad18) -> (no net)
- A1 pad 19: /analog_light -> /220_led
- A1 pad 23: /220_led -> /SCL
- A1 pad 24: /SCL -> /SDA
- A1 pad 25: /SDA -> /analog_light
- A1 pad 26: /sig_unlock -> /sig_220v
- A1 pad 27: /v5 -> (no net)
- A1 pad 28: Net-(A1-Pad28) -> (no net)
- A1 pad 3: Net-(A1-Pad3) -> (no net)
- J1 pad 2: Net-(J1-Pad2) -> (no net)
- J2 pad 5: Net-(J2-Pad5) -> (no net)
- J3 pad 10: Net-(J3-Pad10) -> (no net)
- J3 pad 7: Net-(J3-Pad7) -> (no net)
- J3 pad 8: Net-(J3-Pad8) -> (no net)
- J3 pad 9: Net-(J3-Pad9) -> (no net)
- J5 pad 1: Net-(J5-Pad1) -> (no net)
- J5 pad 2: Net-(J5-Pad2) -> (no net)
- J6 pad 1: /TX -> /RX
- J6 pad 2: /RX -> /TX
- J7 pad 2: Net-(J7-Pad2) -> (no net)
- J9 pad 1: /power_5v -> /door_gnd
- J9 pad 2: /power_eis -> /220_avail
- R18 pad 2: /sig_5v -> /sig_radio
- U2 pad 10: Net-(U2-Pad10) -> (no net)
- U2 pad 7: Net-(U2-Pad7) -> (no net)
- U2 pad 8: Net-(U2-Pad8) -> (no net)
- U2 pad 9: Net-(U2-Pad9) -> (no net)
Routing:
- net /GND: track 363.5 -> 436.2 mm, vias 5 -> 9
- net /220_led: track 67.9 -> 24.3 mm
- net /sig_220v: track 92.3 -> 50.1 mm, vias 2 -> 4
- net /sig_unlock: track 106.2 -> 146.1 mm, vias 6 -> 5
- net /RX: track 107.1 -> 74.5 mm
- net /sig_radio: track 55.4 -> 87.7 mm, vias 2 -> 3
- net /TX: track 96.0 -> 79.3 mm
- net /sig_horn: track 103.0 -> 117.7 mm
- net /analog_light: track 20.1 -> 31.9 mm, vias 1 -> 0
- net /sig_lock: track 102.7 -> 110.7 mm, vias 1 -> 2
- net /inp_gnd: track 172.1 -> 165.8 mm
- net /SDA: track 35.3 -> 29.5 mm, vias 1 -> 0
- net /sig_b: track 194.2 -> 188.8 mm
- net Net-(D8-Pad2): track 0.00 -> 4.83 mm
- net Net-(D6-Pad2): track 0.00 -> 3.92 mm
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- added copper zone on F.Cu, net /GND
- added copper zone on B.Cu, net /VDD
Other:
- board text added: "+12V"
- board text added: "+12V unfused"
- board text added: "GND"
- board text added: "PUFFIS BRAIN ANDIEH V.0.4 (02/2019)"
- board text removed: "12V no fuse | 12V | GND"
- board text removed: "PUFFIS BRAIN ANDIEH V.0.3 (12/2018)"
