File: schematic/car-control/car-control.sch (KiCad schematic (older format))
At the start: 43 parts, among them J1 RGBW Sitzbank, J10 Misc Conn, J2 RGBW Hutablage, J3 RPi Front #1, J4 RPi Front #2, J5 Touch Panel, J6 Alarm Control, J7 RGBW Universell 1, J8 Power_Conn, J9 Sig_in_out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

Commit message: i really have no glue what i have done since the last checkin
Parts:
- removed J9: Sig_in_out, TerminalBlock_Phoenix:TerminalBlock_Phoenix_MKDS-1,5-8-5.08_1x08_P5.08mm_Horizontal, symbol Screw_Terminal_01x07
- added D10: unlock, led:LED_D3.0mm_Clear, symbol LED
- added D6: horn, led:LED_D3.0mm_Clear, symbol LED
- added D8: act_5v, led:LED_D3.0mm_Clear, symbol LED
- added D9: lock, led:LED_D3.0mm_Clear, symbol LED
- added J11: Sig_out, TerminalBlock_Phoenix:TerminalBlock_Phoenix_MKDS-1,5-4-5.08_1x04_P5.08mm_Horizontal, symbol Screw_Terminal_01x04
- added J9: Sig_in, TerminalBlock_Phoenix:TerminalBlock_Phoenix_MKDS-1,5-2-5.08_1x02_P5.08mm_Horizontal, symbol Screw_Terminal_01x02
- added R19, R20, R21, R22: 220, Resistor_THT:R_Axial_DIN0207_L6.3mm_D2.5mm_P10.16mm_Horizontal, symbol R
- D1, D2, D3, D4, D5: footprint led:LED_D5.0mm_Clear -> led:LED_D3.0mm_Clear
- D7: value act_5v -> radio; footprint led:LED_D5.0mm_Clear -> led:LED_D3.0mm_Clear
Connections:
- net 220_avail: now also J9.2 (Pin_2)
- net 220_led: now also A1.19 (A0); no longer A1.23 (A4)
- net GND: now also D10.1 (K), D6.1 (K), D8.1 (K), D9.1 (K)
- net RX: now also J6.1 (Pin_1); no longer J6.2 (Pin_2)
- net SCL: now also A1.23 (A4); no longer A1.24 (A5)
- net SDA: now also A1.24 (A5); no longer A1.25 (A6)
- net TX: now also J6.2 (Pin_2); no longer J6.1 (Pin_1)
- net analog_light: now also A1.25 (A6); no longer A1.19 (A0)
- net door_gnd: now also J9.1 (Pin_1)
- net lock_car: now also J11.3 (Pin_3)
- net power_5v: now also J11.1 (Pin_1)
- net power_eis: now also J11.2 (Pin_2)
- net sig_220v: now also A1.26 (A7); no longer A1.14 (D11)
- net sig_5v: now also R20.2; no longer R18.2
- net sig_horn: now also R19.2
- net sig_lock: now also R21.2
- net sig_radio: now also R18.2
- net sig_unlock: now also A1.14 (D11), R22.2; no longer A1.26 (A7)
- net unlock_car: now also J11.4 (Pin_4)
- new net: D8.2 (A), R20.1
- new net: D6.2 (A), R19.1
- new net: D9.2 (A), R21.1
- new net: D10.2 (A), R22.1
- no-connect marks 14 -> 13
Other:
- moved on the sheet: D5, D7, R16, R18
Changed lines of the file:
@@
 Text Notes 6800 4800 0    60   ~ 0
 Alarm Control
+Text Label 6850 4950 2    60   ~ 0
+RX
 Text Label 7350 4950 0    60   ~ 0
-RX
-Text Label 6850 4950 2    60   ~ 0
 TX
 Text Label 6850 5050 2    60   ~ 0
@@
 Text Label 6850 4050 2    60   ~ 0
 SDA
+Text Label 5650 4100 0    60   ~ 0
+SCL
 Text Label 5650 4200 0    60   ~ 0
-SCL
-Text Label 5650 4300 0    60   ~ 0
 SDA
 Text Label 4650 3300 2    60   ~ 0
@@
 Text Label 4650 4100 2    60   ~ 0
 sig_lock
-Text Label 4650 4200 2    60   ~ 0
+Text Label 5650 4400 0    60   ~ 0
 sig_220v
 Text Label 4650 4300 2    60   ~ 0
@@
 Text Label 4650 4400 2    60   ~ 0
 sig_5v
-Text Label 5650 3700 0    60   ~ 0
+Text Label 5650 4300 0    60   ~ 0
 analog_light
 Text Label 7350 4150 0    60   ~ 0
@@
 Text Label 9850 3850 2    60   ~ 0
 inp_12v_unfused
-$Comp
-L Screw_Terminal_01x07 J9
-U 1 1 5C12F7E7
-P 9550 4900
-F 0 "J9" H 9550 5000 50  0000 C CNN
-F 1 "Sig_in_out" H 9550 4450 50  0000 C CNN
-F 2 "TerminalBlock_Phoenix:TerminalBlock_Phoenix_MKDS-1,5-8-5.08_1x08_P5.08mm_Horizontal" H 9550 4900 50  0001 C CNN
-F 3 "" H 9550 4900 50  0001 C CNN
-	1    9550 4900
-	-1   0    0    1
-$EndComp
 Text Label 9750 4600 0    60   ~ 0
 220_avail
 Text Label 9750 4700 0    60   ~ 0
 door_gnd
-Text Label 9750 5100 0    60   ~ 0
+Text Label 9750 5300 0    60   ~ 0
 power_eis
+Text Label 9750 5400 0    60   ~ 0
+power_5v
 Text Label 9750 5200 0    60   ~ 0
-power_5v
-Text Label 9750 5000 0    60   ~ 0
 lock_car
 NoConn ~ 2000 3850
@@
 Text Label 7350 4350 0    60   ~ 0
 220_led
-Text Label 5650 4100 0    60   ~ 0
+Text Label 5650 3700 0    60   ~ 0
 220_led
 Text Label 5350 1100 2    60   ~ 0
@@
 F 0 "D1" H 3250 3100 50  0000 C CNN
 F 1 "red" H 3250 2900 50  0000 C CNN
-F 2 "led:LED_D5.0mm_Clear" H 3250 3000 50  0001 C CNN
+F 2 "led:LED_D3.0mm_Clear" H 3250 3000 50  0001 C CNN
 F 3 "" H 3250 3000 50  0001 C CNN
 	1    3250 3000
@@
 F 0 "D2" H 3250 3400 50  0000 C CNN
 F 1 "green" H 3250 3200 50  0000 C CNN
-F 2 "led:LED_D5.0mm_Clear" H 3250 3300 50  0001 C CNN
+F 2 "led:LED_D3.0mm_Clear" H 3250 3300 50  0001 C CNN
 F 3 "" H 3250 3300 50  0001 C CNN
 	1    3250 3300
@@
 F 0 "D3" H 3250 3700 50  0000 C CNN
 F 1 "blue" H 3250 3500 50  0000 C CNN
-F 2 "led:LED_D5.0mm_Clear" H 3250 3600 50  0001 C CNN
+F 2 "led:LED_D3.0mm_Clear" H 3250 3600 50  0001 C CNN
 F 3 "" H 3250 3600 50  0001 C CNN
 	1    3250 3600
@@
 F 0 "D4" H 3250 4000 50  0000 C CNN
 F 1 "white" H 3250 3800 50  0000 C CNN
-F 2 "led:LED_D5.0mm_Clear" H 3250 3900 50  0001 C CNN
+F 2 "led:LED_D3.0mm_Clear" H 3250 3900 50  0001 C CNN
 F 3 "" H 3250 3900 50  0001 C CNN
 	1    3250 3900
@@
 L LED D5
 U 1 1 5C1D3F0A
-P 7350 950
-F 0 "D5" H 7350 1050 50  0000 C CNN
-F 1 "act_eis" H 7350 850 50  0000 C CNN
-F 2 "led:LED_D5.0mm_Clear" H 7350 950 50  0001 C CNN
-F 3 "" H 7350 950 50  0001 C CNN
-	1    7350 950
-	1    0    0    -1
-$EndComp
-Text Label 7200 950  2    60   ~ 0
+P 7300 1100
+F 0 "D5" H 7300 1200 50  0000 C CNN
+F 1 "act_eis" H 7300 1000 50  0000 C CNN
+F 2 "led:LED_D3.0mm_Clear" H 7300 1100 50  0001 C CNN
+F 3 "" H 7300 1100 50  0001 C CNN
+	1    7300 1100
+	1    0    0    -1
+$EndComp
+Text Label 7150 1100 2    60   ~ 0
 GND
 $Comp
 L R R16
 U 1 1 5C1D3F12
-P 7650 950
-F 0 "R16" V 7730 950 50  0000 C CNN
-F 1 "220" V 7650 950 50  0000 C CNN
-F 2 "Resistor_THT:R_Axial_DIN0207_L6.3mm_D2.5mm_P10.16mm_Horizontal" V 7580 950 50  0001 C CNN
-F 3 "" H 7650 950 50  0001 C CNN
-	1    7650 950
-	0    -1   -1   0
-$EndComp
-Text Label 7800 950  0    60   ~ 0
+P 7600 1100
+F 0 "R16" V 7680 1100 50  0000 C CNN
+F 1 "220" V 7600 1100 50  0000 C CNN
+F 2 "Resistor_THT:R_Axial_DIN0207_L6.3mm_D2.5mm_P10.16mm_Horizontal" V 7530 1100 50  0001 C CNN
+F 3 "" H 7600 1100 50  0001 C CNN
+	1    7600 1100
+	0    -1   -1   0
+$EndComp
+Text Label 7750 1100 0    60   ~ 0
 sig_eis
 $Comp
 L LED D7
 U 1 1 5C1D4636
-P 7350 1550
-F 0 "D7" H 7350 1650 50  0000 C CNN
-F 1 "act_5v" H 7350 1450 50  0000 C CNN
-F 2 "led:LED_D5.0mm_Clear" H 7350 1550 50  0001 C CNN
-F 3 "" H 7350 1550 50  0001 C CNN
-	1    7350 1550
-	1    0    0    -1
-$EndComp
-Text Label 7200 1550 2    60   ~ 0
+P 7300 1700
+F 0 "D7" H 7300 1800 50  0000 C CNN
+F 1 "radio" H 7300 1600 50  0000 C CNN
+F 2 "led:LED_D3.0mm_Clear" H 7300 1700 50  0001 C CNN
+F 3 "" H 7300 1700 50  0001 C CNN
+	1    7300 1700
+	1    0    0    -1
+$EndComp
+Text Label 7150 1700 2    60   ~ 0
 GND
 $Comp
 L R R18
 U 1 1 5C1D463E
-P 7650 1550
-F 0 "R18" V 7730 1550 50  0000 C CNN
-F 1 "220" V 7650 1550 50  0000 C CNN
-F 2 "Resistor_THT:R_Axial_DIN0207_L6.3mm_D2.5mm_P10.16mm_Horizontal" V 7580 1550 50  0001 C CNN
-F 3 "" H 7650 1550 50  0001 C CNN
-	1    7650 1550
-	0    -1   -1   0
-$EndComp
-Text Label 7800 1550 0    60   ~ 0
-sig_5v
-Text Label 5650 4400 0    60   ~ 0
+P 7600 1700
+F 0 "R18" V 7680 1700 50  0000 C CNN
+F 1 "220" V 7600 1700 50  0000 C CNN
+F 2 "Resistor_THT:R_Axial_DIN0207_L6.3mm_D2.5mm_P10.16mm_Horizontal" V 7530 1700 50  0001 C CNN
+F 3 "" H 7600 1700 50  0001 C CNN
+	1    7600 1700
+	0    -1   -1   0
+$EndComp
+Text Label 7750 1700 0    60   ~ 0
+sig_radio
+Text Label 4650 4200 2    60   ~ 0
 sig_unlock
 Text Label 4450 1800 2    60   ~ 0
@@
 Wire Wire Line
 	5650 1400 5650 1300
-Text Label 9750 4900 0    60   ~ 0
+Text Label 9750 5100 0    60   ~ 0
 unlock_car
 Text Label 9600 2400 2    60   ~ 0
@@
 	0    1    1    0
 $EndComp
-NoConn ~ 9750 4800
 NoConn ~ 7350 2750
 NoConn ~ 7350 2850
@@
 NoConn ~ 7350 4450
 NoConn ~ 6850 4450
+$Comp
+L Screw_Terminal_01x02 J9
+U 1 1 5C48F76D
+P 9550 4700
+F 0 "J9" H 9550 4800 50  0000 C CNN
+F 1 "Sig_in" H 9550 4500 50  0000 C CNN
+F 2 "TerminalBlock_Phoenix:TerminalBlock_Phoenix_MKDS-1,5-2-5.08_1x02_P5.08mm_Horizontal" H 9550 4700 50  0001 C CNN
+F 3 "" H 9550 4700 50  0001 C CNN
+	1    9550 4700
+	-1   0    0    1
+$EndComp
+$Comp
+L Screw_Terminal_01x04 J11
+U 1 1 5C48F81E
+P 9550 5300
+F 0 "J11" H 9550 5500 50  0000 C CNN
+F 1 "Sig_out" H 9550 5000 50  0000 C CNN
+F 2 "TerminalBlock_Phoenix:TerminalBlock_Phoenix_MKDS-1,5-4-5.08_1x04_P5.08mm_Horizontal" H 9550 5300 50  0001 C CNN
+F 3 "" H 9550 5300 50  0001 C CNN
+	1    9550 5300
+	-1   0    0    1
+$EndComp
+$Comp
+L LED D8
+U 1 1 5C48FBDB
+P 7300 1400
+F 0 "D8" H 7300 1500 50  0000 C CNN
+F 1 "act_5v" H 7300 1300 50  0000 C CNN
+F 2 "led:LED_D3.0mm_Clear" H 7300 1400 50  0001 C CNN
+F 3 "" H 7300 1400 50  0001 C CNN
+	1    7300 1400
+	1    0    0    -1
+$EndComp
+Text Label 7150 1400 2    60   ~ 0
+GND
+$Comp
+L R R20
+U 1 1 5C48FBE3
+P 7600 1400
+F 0 "R20" V 7680 1400 50  0000 C CNN
+F 1 "220" V 7600 1400 50  0000 C CNN
+F 2 "Resistor_THT:R_Axial_DIN0207_L6.3mm_D2.5mm_P10.16mm_Horizontal" V 7530 1400 50  0001 C CNN
+F 3 "" H 7600 1400 50  0001 C CNN
+	1    7600 1400
+	0    -1   -1   0
+$EndComp
+Text Label 7750 1400 0    60   ~ 0
+sig_5v
+$Comp
+L LED D6
+U 1 1 5C490421
+P 7300 800
+F 0 "D6" H 7300 900 50  0000 C CNN
+F 1 "horn" H 7300 700 50  0000 C CNN
+F 2 "led:LED_D3.0mm_Clear" H 7300 800 50  0001 C CNN
+F 3 "" H 7300 800 50  0001 C CNN
+	1    7300 800
+	1    0    0    -1
+$EndComp
+Text Label 7150 800  2    60   ~ 0
+GND
+$Comp
+L R R19
+U 1 1 5C490429
+P 7600 800
+F 0 "R19" V 7680 800 50  0000 C CNN
+F 1 "220" V 7600 800 50  0000 C CNN
+F 2 "Resistor_THT:R_Axial_DIN0207_L6.3mm_D2.5mm_P10.16mm_Horizontal" V 7530 800 50  0001 C CNN
+F 3 "" H 7600 800 50  0001 C CNN
+	1    7600 800
+	0    -1   -1   0
+$EndComp
+Text Label 7750 800  0    60   ~ 0
+sig_horn
+$Comp
+L LED D9
+U 1 1 5C490650
+P 8250 2800
+F 0 "D9" H 8250 2900 50  0000 C CNN
+F 1 "lock" H 8250 2700 50  0000 C CNN
+F 2 "led:LED_D3.0mm_Clear" H 8250 2800 50  0001 C CNN
+F 3 "" H 8250 2800 50  0001 C CNN
+	1    8250 2800
+	1    0    0    -1
+$EndComp
+Text Label 8100 2800 2    60   ~ 0
+GND
+$Comp
+L R R21
+U 1 1 5C490658
+P 8550 2800
+F 0 "R21" V 8630 2800 50  0000 C CNN
+F 1 "220" V 8550 2800 50  0000 C CNN
+F 2 "Resistor_THT:R_Axial_DIN0207_L6.3mm_D2.5mm_P10.16mm_Horizontal" V 8480 2800 50  0001 C CNN
+F 3 "" H 8550 2800 50  0001 C CNN
+	1    8550 2800
+	0    -1   -1   0
+$EndComp
+Text Label 8700 2800 0    60   ~ 0
+sig_lock
+$Comp
+L LED D10
+U 1 1 5C490874
+P 8250 3100
+F 0 "D10" H 8250 3200 50  0000 C CNN
+F 1 "unlock" H 8250 3000 50  0000 C CNN
+F 2 "led:LED_D3.0mm_Clear" H 8250 3100 50  0001 C CNN
+F 3 "" H 8250 3100 50  0001 C CNN
+	1    8250 3100
+	1    0    0    -1
+$EndComp
+Text Label 8100 3100 2    60   ~ 0
+GND
+$Comp
+L R R22
+U 1 1 5C49087C
+P 8550 3100
+F 0 "R22" V 8630 3100 50  0000 C CNN
+F 1 "220" V 8550 3100 50  0000 C CNN
+F 2 "Resistor_THT:R_Axial_DIN0207_L6.3mm_D2.5mm_P10.16mm_Horizontal" V 8480 3100 50  0001 C CNN
+F 3 "" H 8550 3100 50  0001 C CNN
+	1    8550 3100
+	0    -1   -1   0
+$EndComp
+Text Label 8700 3100 0    60   ~ 0
+sig_unlock
 $EndSCHEMATC
